Commit message: vibrations roll and z

File: src/dummy_uav/urdf/dummy_uav.urdf.xacro (robot description, xacro)
@@ -16,20 +16,20 @@
     </inertial>
     <visual>
-      <geometry><box size="0.3 0.3 0.1"/></geometry>
+      <geometry><box size="0.2 0.2 0.06"/></geometry>
       <origin xyz="0 0 0" rpy="0 0 0"/>
       <material name="Blue"><color rgba="0 0 1 1"/></material>
     </visual>
-    <collision>
+    <!-- <collision>
       <geometry><box size="0.3 0.3 0.1"/></geometry>
       <origin xyz="0 0 0" rpy="0 0 0"/>
-    </collision>
+    </collision> -->
   </link>
   <!-- Headlight Link -->
-  <link name="headlight_link">
+  <!-- <link name="headlight_link">
     <inertial>
       <mass value="0.01" />
       <origin xyz="0 0 0" rpy="0 0 0" />
       <inertia ixx="1e-6" iyy="1e-6" izz="1e-6" ixy="0" ixz="0" iyz="0" />
-    </inertial>
+    </inertial> -->
     <!-- <visual>
       <geometry><sphere radius="0.02"/></geometry>
@@ -37,12 +37,49 @@
       <material name="White"><color rgba="1 1 1 1"/></material>
     </visual> -->
+  <!-- </link> -->
+  <!-- Bat Link oscillation-->
+  <link name="bat_link">
+    <inertial>
+      <mass value="0.05"/>
+      <origin xyz="0 0 0" rpy="0 0 0"/>
+      <inertia ixx="0.001" iyy="0.001" izz="0.001" ixy="0" ixz="0" iyz="0"/>
+    </inertial>
+    <!-- <visual>
+      <geometry><box size="0.5 0.1 0.05"/></geometry>
+      <origin xyz="0 0 0" rpy="0 0 0"/>
+      <material name="Red"><color rgba="1 0 0 1"/></material>
+    </visual> -->
+    <!-- <collision>
+      <geometry><box size="0.5 0.1 0.05"/></geometry>
+      <origin xyz="0 0 0" rpy="0 0 0"/>
+    </collision> -->
   </link>
-  <joint name="headlight_joint" type="fixed">
+  <!-- Flap Joint -->
+  <joint name="flap_joint" type="revolute">
+    <parent link="bat_link"/>
+    <child link="base_link"/>
+    <origin xyz="0 0 0.05" rpy="0 0 0"/>
+    <axis xyz="1 0 0"/>
+    <limit effort="10" velocity="5.0" lower="-1.5" upper="1.5"/>
+    <dynamics damping="0.1"/>
+  </joint>
+  <!-- Bat Plugin -->
+  <gazebo>
+    <plugin name="flapping_plugin" filename="libflapping_plugin.so">
+      <joint_name>flap_joint</joint_name>
+      <frequency>3.0</frequency>
+      <amplitude>0.1</amplitude>
+      <z_amplitude>0.05</z_amplitude>
+      <z_frequency>1.0</z_frequency>
+    </plugin>
+  </gazebo>
+  <!-- Headlight Joint -->
+  <!-- <joint name="headlight_joint" type="fixed">
     <parent link="base_link"/>
     <child link="headlight_link"/>
     <origin xyz="0.15 0 0.02" rpy="0 0 0"/>
-  </joint>
+  </joint> -->
   <!-- Headlight Gazebo Plugin -->
-  <gazebo reference="headlight_link">
+  <!-- <gazebo reference="headlight_link">
     <light type="spot" name="headlight">
       <pose>0 0 0 0 0 0</pose>
@@ -64,5 +101,5 @@
     </light>
     <material>Gazebo/White</material>
-  </gazebo>
+  </gazebo> -->
   <!-- IMU Link -->
   <link name="imu_link">
@@ -76,5 +113,5 @@
     <parent link="base_link"/>
     <child link="imu_link"/>
-    <origin xyz="0 0 0.05" rpy="0 0 0"/>
+    <origin xyz="0 0 0" rpy="0 0 0"/>
   </joint>
   <gazebo reference="imu_link">
@@ -98,6 +135,26 @@
     </sensor>
   </gazebo>
+  <link name="camera_link">
+    <inertial>
+      <mass value="0.001" />
+      <origin xyz="0 0 0" rpy="0 0 0" />
+      <inertia ixx="1e-6" iyy="1e-6" izz="1e-6" ixy="0" ixz="0" iyz="0" />
+    </inertial>
+  </link>
+  <joint name="camera_joint" type="fixed">
+    <parent link="base_link"/>
+    <child link="camera_link"/>
+    <!-- Adjust these as needed -->
+    <origin xyz="0.05 0 0.05" rpy="0 0 0"/>
+  </joint>
+  <!-- Camera Frame -->
+  <link name="camera_optical_frame"/>
+  <joint name="camera_optical_joint" type="fixed">
+    <parent link="camera_link"/>
+    <child link="camera_optical_frame"/>
+    <origin xyz="0 0 0" rpy="-1.5708 0 -1.5708"/> <!-- Align to OpenCV convention -->
+  </joint>
   <!-- Camera Sensor -->
-  <gazebo reference="base_link">
+  <gazebo reference="camera_link">
     <sensor name="camera_sensor" type="camera">
       <always_on>true</always_on>
@@ -105,7 +162,8 @@
       <visualize>true</visualize>
       <camera>
-        <horizontal_fov>1.39626</horizontal_fov> <!-- ~80 deg -->
+        <horizontal_fov>1.39626</horizontal_fov>  <!--~80 deg -->
+        <!-- <horizontal_fov>2.1472</horizontal_fov> 60 degrees -->
         <image>
-          <width>1280</width>
+          <width>640</width>
           <height>800</height>
           <format>R8G8B8</format>
@@ -113,5 +171,5 @@
         <clip>
           <near>0.1</near>
-          <far>500</far>
+          <far>200</far>
         </clip>
       </camera>
@@ -120,5 +178,5 @@
         <imageTopicName>image_raw</imageTopicName>
         <cameraInfoTopicName>camera_info</cameraInfoTopicName>
-        <frameName>base_link</frameName>
+        <frameName>camera_optical_frame</frameName>
       </plugin>
     </sensor>
